File: sensorboxes-rev2/board/bat_pol_prot.sch (KiCad schematic (older format))
At the start: 24 parts

Commit message: developed more of the schematic for the STM32 + radio. also picked out passives & figured out bidirectional battery polarity checking + reverse polarity protection for the solar panel.
Parts:
- removed BT? (x4): Battery_Cell, symbol Device:Battery_Cell
- removed D? (x2): D, symbol Device:D
- removed Q? (x9): Q_PMOS_DGS, symbol Device:Q_PMOS_DGS
- removed Q? (x2): Q_NMOS_DGS, symbol Device:Q_NMOS_DGS
- removed R? (x5): R, symbol Device:R
- removed U? (x2): TS881xCx, Package_TO_SOT_SMD:SOT-353_SC-70-5, symbol Amplifier_Operational:TS881xCx
Connections:
- net labels removed: GND, VBAT_PROT, VIN, VOUT, VSOLAR_PROT
- wire segments 97 -> 0
Other:
- note removed: "SiP32101"
- note removed: "V_OVERVOLT_THRESH = 4.2V\nV_OK_THRESH = 3.7V\nV_UNDERVOLT_THRESH = 3.2V"
- note removed: "WIP, unknown what to actually put here for a circuit"
