File: sensorboxes-rev2/board/mcu.sch (KiCad schematic (older format))
At the start: 17 parts

Commit message: exposing pins for mcu, added part values for RF section
Parts:
- added JP?: SolderJumper_2_Bridged, symbol Jumper:SolderJumper_2_Bridged
- C? (x4): value C -> 100n
- C? (x2): value C -> 4.3p
Connections:
- net labels added: MCO, PB0, PB1, PB3, PB4, PB5, PB6, PB7, SWCLK, SWDIO, VCP_RX, VCP_TX, ~RST
- wire segments 63 -> 78
Changed lines of the file:
@@
 P 4300 2300
 F 0 "C?" H 4415 2346 50  0000 L CNN
-F 1 "C" H 4415 2255 50  0000 L CNN
+F 1 "100n" H 4415 2255 50  0000 L CNN
 F 2 "" H 4338 2150 50  0001 C CNN
 F 3 "~" H 4300 2300 50  0001 C CNN
@@
 P 1200 1350
 F 0 "C?" H 1315 1396 50  0000 L CNN
-F 1 "C" H 1315 1305 50  0000 L CNN
+F 1 "100n" H 1315 1305 50  0000 L CNN
 F 2 "" H 1238 1200 50  0001 C CNN
 F 3 "~" H 1200 1350 50  0001 C CNN
@@
 P 1600 1350
 F 0 "C?" H 1715 1396 50  0000 L CNN
-F 1 "C" H 1715 1305 50  0000 L CNN
+F 1 "100n" H 1715 1305 50  0000 L CNN
 F 2 "" H 1638 1200 50  0001 C CNN
 F 3 "~" H 1600 1350 50  0001 C CNN
@@
 P 3150 2350
 F 0 "C?" H 3265 2396 50  0000 L CNN
-F 1 "C" H 3265 2305 50  0000 L CNN
+F 1 "100n" H 3265 2305 50  0000 L CNN
 F 2 "" H 3188 2200 50  0001 C CNN
 F 3 "~" H 3150 2350 50  0001 C CNN
@@
 P 1700 4000
 F 0 "C?" H 1815 4046 50  0000 L CNN
-F 1 "C" H 1815 3955 50  0000 L CNN
+F 1 "4.3p" H 1815 3955 50  0000 L CNN
 F 2 "" H 1738 3850 50  0001 C CNN
 F 3 "~" H 1700 4000 50  0001 C CNN
@@
 P 2200 4000
 F 0 "C?" H 2315 4046 50  0000 L CNN
-F 1 "C" H 2315 3955 50  0000 L CNN
+F 1 "4.3p" H 2315 3955 50  0000 L CNN
 F 2 "" H 2238 3850 50  0001 C CNN
 F 3 "~" H 2200 4000 50  0001 C CNN
@@
 Wire Wire Line
 	4450 3800 4600 3800
+Text HLabel 4600 2600 2    50   BiDi ~ 0
+MCO
+Wire Wire Line
+	4450 2600 4600 2600
+Text HLabel 1150 3200 0    50   BiDi ~ 0
+MCO
+Wire Wire Line
+	1300 3200 1150 3200
+$Comp
+L Jumper:SolderJumper_2_Bridged JP?
+U 1 1 5E4E8512
+P 1450 3200
+F 0 "JP?" V 1450 3268 50  0001 L CNN
+F 1 "SolderJumper_2_Bridged" V 1495 3268 50  0001 L CNN
+F 2 "" H 1450 3200 50  0001 C CNN
+F 3 "~" H 1450 3200 50  0001 C CNN
+	1    1450 3200
+	1    0    0    -1
+$EndComp
+Wire Wire Line
+	1600 3200 1700 3200
+Connection ~ 1700 3200
+Text HLabel 4600 2800 2    50   Output ~ 0
+VCP_TX
+Wire Wire Line
+	4600 2800 4450 2800
+Text HLabel 4600 3900 2    50   BiDi ~ 0
+SWDIO
+Wire Wire Line
+	4600 3900 4450 3900
+Text HLabel 4600 4000 2    50   BiDi ~ 0
+SWCLK
+Wire Wire Line
+	4600 4000 4450 4000
+Text HLabel 4600 4100 2    50   Input ~ 0
+VCP_RX
+Wire Wire Line
+	4600 4100 4450 4100
+Text HLabel 3300 3500 0    50   BiDi ~ 0
+PB0
+Wire Wire Line
+	3450 3500 3300 3500
+Text HLabel 3300 3600 0    50   BiDi ~ 0
+PB1
+Wire Wire Line
+	3450 3600 3300 3600
+Text HLabel 3300 3700 0    50   BiDi ~ 0
+PB3
+Wire Wire Line
+	3450 3700 3300 3700
+Text HLabel 3300 3800 0    50   BiDi ~ 0
+PB4
+Wire Wire Line
+	3450 3800 3300 3800
+Text HLabel 3300 3900 0    50   BiDi ~ 0
+PB5
+Wire Wire Line
+	3450 3900 3300 3900
+Text HLabel 3300 4000 0    50   BiDi ~ 0
+PB6
+Wire Wire Line
+	3450 4000 3300 4000
+Text HLabel 3300 4100 0    50   BiDi ~ 0
+PB7
+Wire Wire Line
+	3450 4100 3300 4100
+Text HLabel 2500 2600 0    50   BiDi ~ 0
+~RST
+Wire Wire Line
+	2500 2600 2600 2600
+Connection ~ 2600 2600
 $EndSCHEMATC
