File: sensorboxes-rev2/board/radio.sch (KiCad schematic (older format))
At the start: 30 parts

Commit message: exposing pins for mcu, added part values for RF section
Parts:
- C? (x2): value C -> 1n
- C? (x2): value C -> 39p
- C? (x2): value C -> 3.3p
- C?: value C -> 1u
- C?: value C -> 100n
- C?: value C -> 470n
- C?: value C -> 47n
- C?: value C -> 47p
- C?: value C -> 3p
- C?: value C -> 5.6p
- C? (x2): value C -> 1.8p
- C?: value C -> 2.4p
- L?: value L -> 9.1n
- L?: value L -> 15u
- L?: value L -> 47n
- L?: value L -> 2.5n
- L?: value L -> 4.7n
- L?: value L -> 15n
- R? (x2): value R -> 100
Changed lines of the file:
@@
 $Descr A4 11693 8268
 encoding utf-8
-Sheet 6 8
+Sheet 4 8
 Title ""
 Date ""
@@
 AR Path="/5E4C9109/5E4B6FDC/5E634C23" Ref="C?"  Part="1"
 F 0 "C?" H 3215 1246 50  0000 L CNN
-F 1 "C" H 3215 1155 50  0000 L CNN
+F 1 "1u" H 3215 1155 50  0000 L CNN
 F 2 "" H 3138 1050 50  0001 C CNN
 F 3 "~" H 3100 1200 50  0001 C CNN
@@
 AR Path="/5E4C9109/5E4B6FDC/5E6C6684" Ref="C?"  Part="1"
 F 0 "C?" H 4865 2846 50  0000 L CNN
-F 1 "C" H 4865 2755 50  0000 L CNN
+F 1 "100n" H 4865 2755 50  0000 L CNN
 F 2 "" H 4788 2650 50  0001 C CNN
 F 3 "~" H 4750 2800 50  0001 C CNN
@@
 AR Path="/5E4C9109/5E4B6FDC/5E6D5716" Ref="L?"  Part="1"
 F 0 "L?" V 4300 2350 50  0000 C CNN
-F 1 "L" V 4400 2350 50  0000 C CNN
+F 1 "15u" V 4400 2350 50  0000 C CNN
 F 2 "" H 4450 2350 50  0001 C CNN
 F 3 "~" H 4450 2350 50  0001 C CNN
@@
 AR Path="/5E4C9109/5E4B6FDC/5E711406" Ref="C?"  Part="1"
 F 0 "C?" H 4615 1846 50  0000 L CNN
-F 1 "C" H 4615 1755 50  0000 L CNN
+F 1 "470n" H 4615 1755 50  0000 L CNN
 F 2 "" H 4538 1650 50  0001 C CNN
 F 3 "~" H 4500 1800 50  0001 C CNN
@@
 AR Path="/5E4C9109/5E4B6FDC/5E729E2A" Ref="C?"  Part="1"
 F 0 "C?" H 4565 3696 50  0000 L CNN
-F 1 "C" H 4565 3605 50  0000 L CNN
+F 1 "47n" H 4565 3605 50  0000 L CNN
 F 2 "" H 4488 3500 50  0001 C CNN
 F 3 "~" H 4450 3650 50  0001 C CNN
@@
 AR Path="/5E4C9109/5E4B6FDC/5E729E37" Ref="C?"  Part="1"
 F 0 "C?" H 4915 3696 50  0000 L CNN
-F 1 "C" H 4915 3605 50  0000 L CNN
+F 1 "47p" H 4915 3605 50  0000 L CNN
 F 2 "" H 4838 3500 50  0001 C CNN
 F 3 "~" H 4800 3650 50  0001 C CNN
@@
 AR Path="/5E4C9109/5E4B6FDC/5E746EF5" Ref="L?"  Part="1"
 F 0 "L?" V 4969 3650 50  0000 C CNN
-F 1 "L" V 5060 3650 50  0000 C CNN
+F 1 "47n" V 5060 3650 50  0000 C CNN
 F 2 "" H 5150 3650 50  0001 C CNN
 F 3 "~" H 5150 3650 50  0001 C CNN
@@
 AR Path="/5E4C9109/5E4B6FDC/5E78FDC5" Ref="L?"  Part="1"
 F 0 "L?" V 5319 4300 50  0000 C CNN
-F 1 "L" V 5410 4300 50  0000 C CNN
+F 1 "2.5n" V 5410 4300 50  0000 C CNN
 F 2 "" H 5500 4300 50  0001 C CNN
 F 3 "~" H 5500 4300 50  0001 C CNN
@@
 AR Path="/5E4C9109/5E4B6FDC/5E78FDCB" Ref="C?"  Part="1"
 F 0 "C?" H 5615 3996 50  0000 L CNN
-F 1 "C" H 5615 3905 50  0000 L CNN
+F 1 "3p" H 5615 3905 50  0000 L CNN
 F 2 "" H 5538 3800 50  0001 C CNN
 F 3 "~" H 5500 3950 50  0001 C CNN
@@
 AR Path="/5E4C9109/5E4B6FDC/5E7B7BBC" Ref="C?"  Part="1"
 F 0 "C?" H 5965 4596 50  0000 L CNN
-F 1 "C" H 5965 4505 50  0000 L CNN
+F 1 "5.6p" H 5965 4505 50  0000 L CNN
 F 2 "" H 5888 4400 50  0001 C CNN
 F 3 "~" H 5850 4550 50  0001 C CNN
@@
 AR Path="/5E4C9109/5E4B6FDC/5E7D28F8" Ref="C?"  Part="1"
 F 0 "C?" H 7065 4546 50  0000 L CNN
-F 1 "C" H 7065 4455 50  0000 L CNN
+F 1 "1.8p" H 7065 4455 50  0000 L CNN
 F 2 "" H 6988 4350 50  0001 C CNN
 F 3 "~" H 6950 4500 50  0001 C CNN
@@
 AR Path="/5E4C9109/5E4B6FDC/5E7D2906" Ref="L?"  Part="1"
 F 0 "L?" V 6319 4300 50  0000 C CNN
-F 1 "L" V 6410 4300 50  0000 C CNN
+F 1 "4.7n" V 6410 4300 50  0000 C CNN
 F 2 "" H 6500 4300 50  0001 C CNN
 F 3 "~" H 6500 4300 50  0001 C CNN
@@
 AR Path="/5E4C9109/5E4B6FDC/5E7D290C" Ref="C?"  Part="1"
 F 0 "C?" H 6215 4346 50  0000 L CNN
-F 1 "C" H 6215 4255 50  0000 L CNN
+F 1 "39p" H 6215 4255 50  0000 L CNN
 F 2 "" H 6138 4150 50  0001 C CNN
 F 3 "~" H 6100 4300 50  0001 C CNN
@@
 AR Path="/5E4C9109/5E4B6FDC/5E82CCC6" Ref="L?"  Part="1"
 F 0 "L?" V 1369 3200 50  0000 C CNN
-F 1 "L" V 1460 3200 50  0000 C CNN
+F 1 "15n" V 1460 3200 50  0000 C CNN
 F 2 "" H 1550 3200 50  0001 C CNN
 F 3 "~" H 1550 3200 50  0001 C CNN
@@
 AR Path="/5E4C9109/5E4B6FDC/5E835410" Ref="C?"  Part="1"
 F 0 "C?" H 1665 2846 50  0000 L CNN
-F 1 "C" H 1665 2755 50  0000 L CNN
+F 1 "1.8p" H 1665 2755 50  0000 L CNN
 F 2 "" H 1588 2650 50  0001 C CNN
 F 3 "~" H 1550 2800 50  0001 C CNN
@@
 AR Path="/5E4C9109/5E4B6FDC/5E89EA45" Ref="C?"  Part="1"
 F 0 "C?" H 1665 5746 50  0000 L CNN
-F 1 "C" H 1665 5655 50  0000 L CNN
+F 1 "2.4p" H 1665 5655 50  0000 L CNN
 F 2 "" H 1588 5550 50  0001 C CNN
 F 3 "~" H 1550 5700 50  0001 C CNN
@@
 Wire Wire Line
 	1550 5900 3250 5900
-Text HLabel 3600 6600 0    50   Output ~ 0
+Text HLabel 3600 6600 0    50   BiDi ~ 0
 DIO2
 Wire Wire Line
@@
 P 3850 6600
 F 0 "R?" H 3920 6646 50  0000 L CNN
-F 1 "R" H 3920 6555 50  0000 L CNN
+F 1 "100" H 3920 6555 50  0000 L CNN
 F 2 "" V 3780 6600 50  0001 C CNN
 F 3 "~" H 3850 6600 50  0001 C CNN
@@
 P 4100 6850
 F 0 "C?" H 4215 6896 50  0000 L CNN
-F 1 "C" H 4215 6805 50  0000 L CNN
+F 1 "1n" H 4215 6805 50  0000 L CNN
 F 2 "" H 4138 6700 50  0001 C CNN
 F 3 "~" H 4100 6850 50  0001 C CNN
@@
 AR Path="/5E4C9109/5E4B6FDC/5E4F896B" Ref="C?"  Part="1"
 F 0 "C?" H 4915 5746 50  0000 L CNN
-F 1 "C" H 4915 5655 50  0000 L CNN
+F 1 "39p" H 4915 5655 50  0000 L CNN
 F 2 "" H 4838 5550 50  0001 C CNN
 F 3 "~" H 4800 5700 50  0001 C CNN
@@
 AR Path="/5E4C9109/5E4B6FDC/5E4FE968" Ref="C?"  Part="1"
 F 0 "C?" H 5165 5996 50  0000 L CNN
-F 1 "C" H 5165 5905 50  0000 L CNN
+F 1 "3.3p" H 5165 5905 50  0000 L CNN
 F 2 "" H 5088 5800 50  0001 C CNN
 F 3 "~" H 5050 5950 50  0001 C CNN
@@
 AR Path="/5E4C9109/5E4B6FDC/5E5053B8" Ref="L?"  Part="1"
 F 0 "L?" V 5169 5700 50  0000 C CNN
-F 1 "L" V 5260 5700 50  0000 C CNN
+F 1 "9.1n" V 5260 5700 50  0000 C CNN
 F 2 "" H 5350 5700 50  0001 C CNN
 F 3 "~" H 5350 5700 50  0001 C CNN
@@
 AR Path="/5E4C9109/5E4B6FDC/5E50E647" Ref="C?"  Part="1"
 F 0 "C?" H 5715 5996 50  0000 L CNN
-F 1 "C" H 5715 5905 50  0000 L CNN
+F 1 "3.3p" H 5715 5905 50  0000 L CNN
 F 2 "" H 5638 5800 50  0001 C CNN
 F 3 "~" H 5600 5950 50  0001 C CNN
@@
 P 6850 5750
 F 0 "C?" H 6965 5796 50  0000 L CNN
-F 1 "C" H 6965 5705 50  0000 L CNN
+F 1 "1n" H 6965 5705 50  0000 L CNN
 F 2 "" H 6888 5600 50  0001 C CNN
 F 3 "~" H 6850 5750 50  0001 C CNN
@@
 P 7100 5500
 F 0 "R?" H 7170 5546 50  0000 L CNN
-F 1 "R" H 7170 5455 50  0000 L CNN
+F 1 "100" H 7170 5455 50  0000 L CNN
 F 2 "" V 7030 5500 50  0001 C CNN
 F 3 "~" H 7100 5500 50  0001 C CNN
