File: sensorboxes-rev2/board/pwr_mgr.sch (KiCad schematic (older format))
At the start: 8 parts

Commit message: developed more of the schematic for the STM32 + radio. also picked out passives & figured out bidirectional battery polarity checking + reverse polarity protection for the solar panel.
Parts:
- added RV?: 1M, symbol Device:R_POT
- C? (x2): value C -> 4.7u
- C?: value C -> 100n
- C?: value C -> 10n
- L?: value L -> 22u
- R?: value R -> 8.2M
- R?: value R -> 2.7
Connections:
- net labels removed: OK_THRESH_H, OK_THRESH_L, OVERVOLT_THRESH, UNDERVOLT_THRESH
- wire segments 40 -> 37
Other:
- moved on the sheet: R?
