File: sensorboxes-rev2/board/board.sch (KiCad schematic (older format))
At the start: 28 parts

Commit message: new schematic for real now. modeled after the feather m0 lora to a T
Parts:
- removed C? (x10): C, symbol Device:C
- removed D?: LED, symbol Device:LED
- removed J?: Conn_ARM_JTAG_SWD_10, symbol Connector:Conn_ARM_JTAG_SWD_10
- removed JP? (x4): Jumper, symbol Device:Jumper
- removed L? (x2): L, symbol Device:L
- removed Q?: Q_NMOS_DGS, symbol Device:Q_NMOS_DGS
- removed R? (x6): R, symbol Device:R
- removed SW?: SW_Push, symbol Switch:SW_Push
- removed U?: ATSAML21J18B-AUT, Package_QFP:TQFP-64_10x10mm_P0.5mm, symbol MCU_Microchip_SAML:ATSAML21J18B-AUT
- removed Y?: Crystal_GND3, symbol Device:Crystal_GND3
- added AE1: Antenna, symbol Device:Antenna
- added C1, C3, C6: 10u, symbol Device:C
- added C10, C11, C4, C5, C8, C9: 100n, symbol Device:C
- added C2: 1u, symbol Device:C
- added C7: 2.2u, symbol Device:C
- added D1: D_Schottky, symbol Device:D_Schottky
- added D2, D3, D4: LED, symbol Device:LED
- added FB1: Ferrite_Bead, symbol Device:Ferrite_Bead
- added J1: USB_B_Micro, symbol Connector:USB_B_Micro
- added J2: Conn_01x12, symbol Connector_Generic:Conn_01x12
- added J3: Conn_01x02, symbol Connector_Generic:Conn_01x02
- added J4: Conn_ARM_JTAG_SWD_10, symbol Connector:Conn_ARM_JTAG_SWD_10
- added J5: Conn_01x11, symbol Connector_Generic:Conn_01x11
- added J6: Conn_01x03, symbol Connector_Generic:Conn_01x03
- added L1: 10u, symbol Device:L
- added Q1, Q2: Q_PMOS_GDS, symbol Device:Q_PMOS_GDS
- added R1, R6, R7: 1k, symbol Device:R
- added R2, R3: 330, symbol Device:R
- added R4: 10k, symbol Device:R
- added R5: 4, symbol Device:R
- added R8: 2.2k, symbol Device:R
- added SW1: SW_Push, symbol Switch:SW_Push
- added U1: ATSAML21E18B-AUT, Package_QFP:TQFP-32_7x7mm_P0.8mm, symbol MCU_Microchip_SAML:ATSAML21E18B-AUT
- added U2: MCP1812A, symbol sensenet_board_part_subs:MCP1812
- added U3: LTC4070, symbol sensenet_board_part_subs:LTC4070
- added U4: RFM69HCW, symbol RF_Module:RFM69HCW
Connections:
- net labels added: +3V3, +BATT, D+, D-, D0, D1, D10, D11, D12, D13, D14, D15, D16, D18, D19, D2, D20, D21, D22, D23, D3, D4, D5, D6, D7, D8, D9, MISO, MOSI, RESET, SCK, SWCLK, SWDIO, VBAT_PROT, VBUS
- net labels removed: PERIPH_VDDIN, SAML21_RESET, SAML21_SWDCLK, SAML21_SWDIO, SAML21_VDDIN
- wire segments 110 -> 193
- no-connect marks 28 -> 0
Other:
- note added: "400 = 5 mA\n40 = 50 mA\n4 = 500 mA"
- note added: "ADJ = GND for 4V float \nADJ = NC for 4.1V float \nADJ = VCC for 4.2V float"
- note added: "Battery Charging and Battery Disconnect"
- note added: "Breakouts"
- note added: "Core"
- note added: "Need to pick the pins to hardwire to the radio, \nor just expose them externally"
- note added: "Power Supply (and Related Connectors)"
- note added: "Reset Switch"
- note added: "User LED"
- note removed: "SAML21_VDDIN is VCC_MCU_P3V3 e.g. current going solely to the chip.\n"
- note removed: "VCC_TARGET is power to peripherals, hardware modules that are NOT the MCU."
- note removed: "Would like the power for peripherals to be selectable and separate from the core."
- note removed: "sourced from regulator to MCU"

Commit message: updated schematic with more specific parts
Parts:
- added JP? (x3): Jumper_NC_Small, symbol Device:Jumper_NC_Small
- D1: value D_Schottky -> MBR120
- FB1: value Ferrite_Bead -> FBMH3216HM221NT
- J5: symbol Connector_Generic:Conn_01x11 -> Connector_Generic:Conn_01x09
- Q1, Q2: value Q_PMOS_GDS -> Si3469DV
- R5: value 4 -> 4.7
Connections:
- net labels added: D17, RFM_DIO1, RFM_DIO2, RFM_DIO3, RFM_DIO5, RFM_IRQ, RFM_RST, SERCOM1_PAD0, SERCOM1_PAD1, SERCOM1_PAD2, SERCOM1_PAD3
- net labels removed: D21, D22, D23, MISO, MOSI, SCK
- wire segments 193 -> 197
Other:
- note added: "Battery temp monitoring not used,\ncan't put the IC near the batteries"
- note added: "Breakouts & Connectors"
- note added: "Example SPI pin mapping requires \nDOPO = 0x1 and DIPO = 0x1\n\nCauses SCK = PAD3, MOSI = PAD2, \nMISO = PAD1, and SS = PAD0"
- note added: "External oscillators may be attached to\nPA00 & PA01 or PA14 & PA15\n"
- note added: "LED can be\ndisconnected to \navoid power draw \nif not needed"
- note added: "Optional status LEDs \nfor battery state can \nbe disconnected?"
- note added: "Radio"
- note added: "SPI Pin Config Limitations:\nMOSI = PAD0, PAD2, PAD3\nMISO = ANY\nSCK = PAD1, PAD3\nSS = ANY"
- note added: "Select Ferrite Bead with \nZ = 50 at 20 MHz and\nZ= 220 at 100 MHz"
- note added: "Slight conflict:\n\nCurrent radio pins also support I2C which REQUIRE \nan external pullup"
- note removed: "Breakouts"
- note removed: "Need to pick the pins to hardwire to the radio, \nor just expose them externally"
- moved on the sheet: C11, R5, R6, R7, R8

Commit message: added TP1, TP2, TP3 to support verification of input power supplies. not sure of any other suitable test point locations aside from communication points like the debug headers, etc. Also added JP4, JP5, JP6 which enable measuring of current out of the whole 3.3V supply, current to the core, and current to the radio. I think that only JP4 is particularly useful though, imho.
Parts:
- added JP4, JP5, JP6: Jumper_NC_Small, symbol Device:Jumper_NC_Small
- added TP? (x3): TestPoint, symbol Connector:TestPoint
- gave numbers to parts that had none: 3
Connections:
- wire segments 197 -> 205
Other:
- moved on the sheet: C7
Changed lines of the file:
@@
 L Connector_Generic:Conn_01x02 J3
 U 1 1 5EB16A74
-P 5600 1350
-F 0 "J3" H 5680 1342 50  0000 L CNN
-F 1 "Conn_01x02" H 5680 1251 50  0000 L CNN
-F 2 "" H 5600 1350 50  0001 C CNN
-F 3 "~" H 5600 1350 50  0001 C CNN
-	1    5600 1350
+P 5300 1350
+F 0 "J3" H 5380 1342 50  0000 L CNN
+F 1 "Conn_01x02" H 5380 1251 50  0000 L CNN
+F 2 "" H 5300 1350 50  0001 C CNN
+F 3 "~" H 5300 1350 50  0001 C CNN
+	1    5300 1350
 	-1   0    0    -1
 $EndComp
@@
 L Device:C C7
 U 1 1 5EB2561F
-P 3200 1800
-F 0 "C7" H 3315 1846 50  0000 L CNN
-F 1 "2.2u" H 3315 1755 50  0000 L CNN
-F 2 "" H 3238 1650 50  0001 C CNN
-F 3 "~" H 3200 1800 50  0001 C CNN
-	1    3200 1800
-	1    0    0    -1
-$EndComp
-Wire Wire Line
-	3200 2050 3200 1950
+P 3450 1800
+F 0 "C7" H 3565 1846 50  0000 L CNN
+F 1 "2.2u" H 3565 1755 50  0000 L CNN
+F 2 "" H 3488 1650 50  0001 C CNN
+F 3 "~" H 3450 1800 50  0001 C CNN
+	1    3450 1800
+	1    0    0    -1
+$EndComp
+Wire Wire Line
+	3450 2050 3450 1950
 $Comp
 L power:GND #PWR0104
 U 1 1 5EB25E68
-P 3200 2050
-F 0 "#PWR0104" H 3200 1800 50  0001 C CNN
-F 1 "GND" H 3205 1877 50  0000 C CNN
-F 2 "" H 3200 2050 50  0001 C CNN
-F 3 "" H 3200 2050 50  0001 C CNN
-	1    3200 2050
-	1    0    0    -1
-$EndComp
-Wire Wire Line
-	3200 1650 3200 1550
-Wire Wire Line
-	3200 1550 3050 1550
+P 3450 2050
+F 0 "#PWR0104" H 3450 1800 50  0001 C CNN
+F 1 "GND" H 3455 1877 50  0000 C CNN
+F 2 "" H 3450 2050 50  0001 C CNN
+F 3 "" H 3450 2050 50  0001 C CNN
+	1    3450 2050
+	1    0    0    -1
+$EndComp
 $Comp
 L power:+3V3 #PWR0105
 U 1 1 5EB26537
-P 3200 1050
-F 0 "#PWR0105" H 3200 900 50  0001 C CNN
-F 1 "+3V3" H 3215 1223 50  0000 C CNN
-F 2 "" H 3200 1050 50  0001 C CNN
-F 3 "" H 3200 1050 50  0001 C CNN
-	1    3200 1050
-	1    0    0    -1
-$EndComp
-Connection ~ 3200 1550
-Wire Wire Line
-	3200 1050 3200 1550
+P 3450 1050
+F 0 "#PWR0105" H 3450 900 50  0001 C CNN
+F 1 "+3V3" H 3465 1223 50  0000 C CNN
+F 2 "" H 3450 1050 50  0001 C CNN
+F 3 "" H 3450 1050 50  0001 C CNN
+	1    3450 1050
+	1    0    0    -1
+$EndComp
 $Comp
 L power:+BATT #PWR0106
 U 1 1 5EB36FFE
-P 5900 1250
-F 0 "#PWR0106" H 5900 1100 50  0001 C CNN
-F 1 "+BATT" H 5915 1423 50  0000 C CNN
-F 2 "" H 5900 1250 50  0001 C CNN
-F 3 "" H 5900 1250 50  0001 C CNN
-	1    5900 1250
-	1    0    0    -1
-$EndComp
-Wire Wire Line
-	5900 1250 5900 1350
-Wire Wire Line
-	5900 1350 5800 1350
+P 5600 1250
+F 0 "#PWR0106" H 5600 1100 50  0001 C CNN
+F 1 "+BATT" H 5615 1423 50  0000 C CNN
+F 2 "" H 5600 1250 50  0001 C CNN
+F 3 "" H 5600 1250 50  0001 C CNN
+	1    5600 1250
+	1    0    0    -1
+$EndComp
+Wire Wire Line
+	5600 1250 5600 1350
+Wire Wire Line
+	5600 1350 5500 1350
 $Comp
 L power:GND #PWR0107
 U 1 1 5EB38662
-P 5900 1550
-F 0 "#PWR0107" H 5900 1300 50  0001 C CNN
-F 1 "GND" H 5905 1377 50  0000 C CNN
-F 2 "" H 5900 1550 50  0001 C CNN
-F 3 "" H 5900 1550 50  0001 C CNN
-	1    5900 1550
-	1    0    0    -1
-$EndComp
-Wire Wire Line
-	5900 1550 5900 1450
-Wire Wire Line
-	5900 1450 5800 1450
+P 5600 1550
+F 0 "#PWR0107" H 5600 1300 50  0001 C CNN
+F 1 "GND" H 5605 1377 50  0000 C CNN
+F 2 "" H 5600 1550 50  0001 C CNN
+F 3 "" H 5600 1550 50  0001 C CNN
+	1    5600 1550
+	1    0    0    -1
+$EndComp
+Wire Wire Line
+	5600 1550 5600 1450
+Wire Wire Line
+	5600 1450 5500 1450
 Wire Wire Line
 	4500 1200 4400 1200
-Wire Wire Line
-	4500 1100 4500 1200
-$Comp
-L power:VBUS #PWR0108
-U 1 1 5EB39218
-P 4500 1100
-F 0 "#PWR0108" H 4500 950 50  0001 C CNN
-F 1 "VBUS" H 4515 1273 50  0000 C CNN
-F 2 "" H 4500 1100 50  0001 C CNN
-F 3 "" H 4500 1100 50  0001 C CNN
-	1    4500 1100
-	1    0    0    -1
-$EndComp
 $Comp
 L Connector:USB_B_Micro J1
@@
 L power:+3V3 #PWR0115
 U 1 1 5EC4060F
-P 9600 2750
-F 0 "#PWR0115" H 9600 2600 50  0001 C CNN
-F 1 "+3V3" H 9615 2923 50  0000 C CNN
-F 2 "" H 9600 2750 50  0001 C CNN
-F 3 "" H 9600 2750 50  0001 C CNN
-	1    9600 2750
+P 10000 2750
+F 0 "#PWR0115" H 10000 2600 50  0001 C CNN
+F 1 "+3V3" H 10015 2923 50  0000 C CNN
+F 2 "" H 10000 2750 50  0001 C CNN
+F 3 "" H 10000 2750 50  0001 C CNN
+	1    10000 2750
 	1    0    0    -1
 $EndComp
@@
 	0    1    1    0
 $EndComp
-Connection ~ 9600 2850
 Wire Wire Line
 	9600 2850 9600 3100
-Wire Wire Line
-	9600 2750 9600 2850
 Wire Wire Line
 	9150 2850 9200 2850
@@
 L power:+3V3 #PWR0124
 U 1 1 5ED4F841
-P 800 3700
-F 0 "#PWR0124" H 800 3550 50  0001 C CNN
-F 1 "+3V3" H 815 3873 50  0000 C CNN
-F 2 "" H 800 3700 50  0001 C CNN
-F 3 "" H 800 3700 50  0001 C CNN
-	1    800  3700
+P 650 3700
+F 0 "#PWR0124" H 650 3550 50  0001 C CNN
+F 1 "+3V3" H 665 3873 50  0000 C CNN
+F 2 "" H 650 3700 50  0001 C CNN
+F 3 "" H 650 3700 50  0001 C CNN
+	1    650  3700
 	1    0    0    -1
 $EndComp
@@
 $EndComp
 Wire Wire Line
-	800  3700 800  3950
-Wire Wire Line
-	800  3950 1050 3950
+	650  3700 650  3950
 $Comp
 L Device:C C2
@@
 Reset Switch
 $Comp
-L Device:Jumper_NC_Small JP?
+L Device:Jumper_NC_Small JP3
 U 1 1 5EB3339C
 P 10200 6150
-F 0 "JP?" V 10154 6224 50  0000 L CNN
+F 0 "JP3" V 10154 6224 50  0000 L CNN
 F 1 "Jumper_NC_Small" V 10245 6224 50  0000 L CNN
 F 2 "" H 10200 6150 50  0001 C CNN
@@
 	10200 5350 10200 5300
 $Comp
-L Device:Jumper_NC_Small JP?
+L Device:Jumper_NC_Small JP1
 U 1 1 5EB3D031
 P 8850 1800
-F 0 "JP?" V 8804 1874 50  0000 L CNN
+F 0 "JP1" V 8804 1874 50  0000 L CNN
 F 1 "Jumper_NC_Small" V 8895 1874 50  0001 L CNN
 F 2 "" H 8850 1800 50  0001 C CNN
@@
 	8950 1800 9150 1800
 $Comp
-L Device:Jumper_NC_Small JP?
+L Device:Jumper_NC_Small JP2
 U 1 1 5EB762B9
 P 9400 1900
-F 0 "JP?" V 9354 1974 50  0000 L CNN
+F 0 "JP2" V 9354 1974 50  0000 L CNN
 F 1 "Jumper_NC_Small" V 9445 1974 50  0001 L CNN
 F 2 "" H 9400 1900 50  0001 C CNN
@@
 Wire Notes Line
 	7800 2500 7800 6550
+$Comp
+L Device:Jumper_NC_Small JP4
+U 1 1 5EB7010A
+P 850 3950
+F 0 "JP4" V 804 4024 50  0000 L CNN
+F 1 "Jumper_NC_Small" V 895 4024 50  0001 L CNN
+F 2 "" H 850 3950 50  0001 C CNN
+F 3 "~" H 850 3950 50  0001 C CNN
+	1    850  3950
+	-1   0    0    1
+$EndComp
+Wire Wire Line
+	950  3950 1050 3950
+Wire Wire Line
+	650  3950 750  3950
+$Comp
+L Device:Jumper_NC_Small JP5
+U 1 1 5EBAAD0E
+P 9800 2850
+F 0 "JP5" V 9754 2924 50  0000 L CNN
+F 1 "Jumper_NC_Small" V 9845 2924 50  0001 L CNN
+F 2 "" H 9800 2850 50  0001 C CNN
+F 3 "~" H 9800 2850 50  0001 C CNN
+	1    9800 2850
+	-1   0    0    1
+$EndComp
+Wire Wire Line
+	9700 2850 9600 2850
+Connection ~ 9600 2850
+Wire Wire Line
+	10000 2750 10000 2850
+Wire Wire Line
+	10000 2850 9900 2850
+Wire Wire Line
+	4500 1100 4500 1200
+$Comp
+L power:VBUS #PWR0108
+U 1 1 5EB39218
+P 4500 1100
+F 0 "#PWR0108" H 4500 950 50  0001 C CNN
+F 1 "VBUS" H 4515 1273 50  0000 C CNN
+F 2 "" H 4500 1100 50  0001 C CNN
+F 3 "" H 4500 1100 50  0001 C CNN
+	1    4500 1100
+	1    0    0    -1
+$EndComp
+$Comp
+L Device:Jumper_NC_Small JP6
+U 1 1 5EBF4F54
+P 3200 1550
+F 0 "JP6" V 3154 1624 50  0000 L CNN
+F 1 "Jumper_NC_Small" V 3245 1624 50  0001 L CNN
+F 2 "" H 3200 1550 50  0001 C CNN
+F 3 "~" H 3200 1550 50  0001 C CNN
+	1    3200 1550
+	-1   0    0    1
+$EndComp
+Wire Wire Line
+	3050 1550 3100 1550
+Wire Wire Line
+	3300 1550 3450 1550
+Connection ~ 3450 1550
+Wire Wire Line
+	3450 1550 3450 1650
+$Comp
+L Connector:TestPoint TP?
+U 1 1 5EC91549
+P 1500 1550
+F 0 "TP?" V 1695 1622 50  0000 C CNN
+F 1 "TestPoint" V 1604 1622 50  0000 C CNN
+F 2 "" H 1700 1550 50  0001 C CNN
+F 3 "~" H 1700 1550 50  0001 C CNN
+	1    1500 1550
+	0    -1   -1   0
+$EndComp
+Wire Wire Line
+	1500 1550 1650 1550
+Connection ~ 1650 1550
+Wire Wire Line
+	3450 1050 3450 1400
+$Comp
+L Connector:TestPoint TP?
+U 1 1 5ECB9E86
+P 3300 1400
+F 0 "TP?" V 3495 1472 50  0000 C CNN
+F 1 "TestPoint" V 3404 1472 50  0000 C CNN
+F 2 "" H 3500 1400 50  0001 C CNN
+F 3 "~" H 3500 1400 50  0001 C CNN
+	1    3300 1400
+	0    -1   -1   0
+$EndComp
+Wire Wire Line
+	3300 1400 3450 1400
+Connection ~ 3450 1400
+Wire Wire Line
+	3450 1400 3450 1550
+$Comp
+L Connector:TestPoint TP?
+U 1 1 5ECD3817
+P 5750 1350
+F 0 "TP?" V 5945 1422 50  0000 C CNN
+F 1 "TestPoint" V 5854 1422 50  0000 C CNN
+F 2 "" H 5950 1350 50  0001 C CNN
+F 3 "~" H 5950 1350 50  0001 C CNN
+	1    5750 1350
+	0    1    1    0
+$EndComp
+Wire Wire Line
+	5750 1350 5600 1350
+Connection ~ 5600 1350
 $EndSCHEMATC

Commit message: added a crystal. dropped the test points from the equation. subbed in RFM95, added some external pullups that have to be 'selected' via a quick blob of solder
Parts:
- removed D2, D3: LED, symbol Device:LED
- removed JP1, JP2, JP4, JP5, JP6: Jumper_NC_Small, symbol Device:Jumper_NC_Small
- removed R6, R7: 1k, symbol Device:R
- removed TP? (x3): TestPoint, symbol Connector:TestPoint
- removed U4: RFM69HCW, symbol RF_Module:RFM69HCW
- added C? (x2): C, symbol Device:C
- added JP?: SolderJumper_2_Open, symbol Jumper:SolderJumper_2_Open
- added R? (x2): 4.7k, symbol Device:R
- added U4: RFM95W-915S2, symbol RF_Module:RFM95W-915S2
- added Y?: MS1V-T1K, symbol Device:Crystal_GND2
- renumbered C8 to C7, C7 to C8, D4 to D2, J3 to J2, J2 to J3, JP3 to JP1, R8 to R6
Connections:
- wire segments 205 -> 200
Other:
- note removed: "Slight conflict:\n\nCurrent radio pins also support I2C which REQUIRE \nan external pullup"

Commit message: added a hierarchical sheet for the core and chose abstracted labels for the pins. reorganized sheet slightly
Parts:
- removed C1, C6: 10u, symbol Device:C
- removed C2: 1u, symbol Device:C
- removed C4, C5, C7: 100n, symbol Device:C
- removed C? (x2): C, symbol Device:C
- removed FB1: FBMH3216HM221NT, symbol Device:Ferrite_Bead
- removed J3: Conn_01x12, symbol Connector_Generic:Conn_01x12
- removed J5: Conn_01x11, symbol Connector_Generic:Conn_01x09
- removed JP1: Jumper_NC_Small, symbol Device:Jumper_NC_Small
- removed JP?: SolderJumper_2_Open, symbol Jumper:SolderJumper_2_Open
- removed L1: 10u, symbol Device:L
- removed R6: 2.2k, symbol Device:R
- removed R? (x2): 4.7k, symbol Device:R
- removed U1: ATSAML21E18B-AUT, Package_QFP:TQFP-32_7x7mm_P0.8mm, symbol MCU_Microchip_SAML:ATSAML21E18B-AUT
- removed Y?: MS1V-T1K, symbol Device:Crystal_GND2
- added J5: Conn_01x06, symbol Connector_Generic:Conn_01x06
- added J6: Conn_01x13, symbol Connector_Generic:Conn_01x13
- added JP1: Jumper_3_Open, symbol Jumper:Jumper_3_Open
- added JP2: Jumper_NC_Small, symbol Device:Jumper_NC_Small
- added R3: 10k, symbol Device:R
- added R5: 2.2k, symbol Device:R
- added TH1: NTHS0402N02N1002F, symbol Device:Thermistor_NTC
- renumbered C3 to C1, C8 to C2, C10 to C3, C11 to C4, C9 to C5, J4 to J1, J1 to J2, J2 to J3, J6 to J4, R5 to R4, R4 to R6, R3 to R7, U2 to U1, U3 to U2, U4 to U3
Connections:
- net labels added: A0, A1, A2, A3, A4, A5, VBAT_CHRG
- net labels removed: D14, D15, D16, D17, D18, D19, D20, RFM_IRQ, RFM_RST, SERCOM1_PAD0, SERCOM1_PAD1, SERCOM1_PAD2, SERCOM1_PAD3
- wire segments 200 -> 157
Other:
- note added: "Analog I/O Header"
- note added: "Cortex Debug Connector"
- note added: "DOPO = 0x1, DIPO = 0x1\n\nSCK = PAD3, MOSI = PAD2,\nMISO = PAD1, SS = PAD0"
- note added: "Digital I/O Header"
- note added: "I2C Pins:\n\nD0, D1\nD6, D7\nD10, D11\n\nSerial Pins (using port function C):\n\nSERCOM0: D0, D1, D2, D3\nSERCOM1: D6, D7, D8, D9\nSERCOM2: D4, D5\nSERCOM3: D10, D11\n\nSerial Pins (using port function D):\n\nSERCOM0: A2, A3, A4, A5\nSERCOM2: D0, D1, D2, D3\nSERCOM3: D6, D7, D8, D9\nSERCOM4: D4, D5\nSERCOM5: D10, D11\n\n"
- note added: "JP2 sets max charge voltage. \n3+2 = 4.2V, 1+2 = 4.0V, NC = 4.1V"
- note removed: "ADJ = GND for 4V float \nADJ = NC for 4.1V float \nADJ = VCC for 4.2V float"
- note removed: "Battery temp monitoring not used,\ncan't put the IC near the batteries"
- note removed: "Example SPI pin mapping requires \nDOPO = 0x1 and DIPO = 0x1\n\nCauses SCK = PAD3, MOSI = PAD2, \nMISO = PAD1, and SS = PAD0"
- note removed: "External oscillators may be attached to\nPA00 & PA01 or PA14 & PA15\n"
- note removed: "Optional status LEDs \nfor battery state can \nbe disconnected?"
- note removed: "SPI Pin Config Limitations:\nMOSI = PAD0, PAD2, PAD3\nMISO = ANY\nSCK = PAD1, PAD3\nSS = ANY"
- note removed: "Select Ferrite Bead with \nZ = 50 at 20 MHz and\nZ= 220 at 100 MHz"
- moved on the sheet: C1, C2, C3, C4, C5, R1, R2, R4, R6, R7
