File: sensorboxes-rev2/board/core.sch (KiCad schematic (older format))
At the start: 14 parts, among them U4 ATSAML21E18B-AUT, Y1 MS1V-T1K

Commit message: changed labeling scheme
Connections:
- net labels added: SERCOM0.0_SPI0_DO, SERCOM0.1_SPI0_SCK, SERCOM0.2_SPI0_SS, SERCOM0.3_SPI0_DI, SERCOM1.0_SPI1_DO, SERCOM1.1_SPI1_SCK, SERCOM1.2_SPI1_SS, SERCOM1.3_SPI1_DI, SERCOM2.2_UART_TX, SERCOM2.3_UART_RX, SERCOM3.0_I2C_SDA, SERCOM3.1_I2C_SCL
- net labels removed: ADC_AIN0, ADC_AIN1, ADC_AIN16, ADC_AIN17, ADC_AIN18, ADC_AIN19, ADC_AIN4, ADC_AIN5, ADC_AIN6, ADC_AIN7, CCL0_IN0, CCL0_IN1, CCL0_IN2, CCL0_OUT, CCL1_IN0, CCL1_IN1, CCL1_IN2, CCL1_OUT1, COMP_AIN0, COMP_AIN1, COMP_AIN2, COMP_AIN3, DAC_VOUT0, DAC_VOUT1, GCLK_IO4, GCLK_IO5, OPAMP_OA_NEG0, OPAMP_OA_OUT0, OPAMP_OA_OUT2, OPAMP_OA_POS0, OPAMP_OA_POS2, PA00, PA01, PA02, PA03, PA04, PA05, PA06, PA07, PA08, PA09, PA10, PA11, PA14, PTC_X0Y6, PTC_X1Y7, PTC_X2Y8, PTC_X3Y9, PTC_Y0, PTC_Y1, PTC_Y4, SERCOM0_PAD0, SERCOM0_PAD1, SERCOM0_PAD2, SERCOM0_PAD3, SERCOM1_PAD0, SERCOM1_PAD1, SERCOM2_PAD0, SERCOM2_PAD1, SERCOM2_PAD2, SERCOM2_PAD3, SERCOM4_PAD2, TCC0_W0, TCC0_W1, TCC0_W2, TCC0_W3, TCC1_W0, TCC1_W1, TCC1_W2, TCC1_W3, TCC2_W0, TCC2_W1, TCC4_W0, TCC4_W1, VREFA, VREFB
- wire segments 220 -> 67
Other:
- note added: "Precondition: All SERCOMS are on Port Function C.\n\nSPI Config (DOPO = 0x0, DIPO = 0x3):\nSCK = PAD1, \nDO = PAD0,\nDI = PAD3, \nSS = PAD2\n\nI2C Config:\nSDA = PAD0,\nSCL = PAD1,\n\nUART Config (RXPO = 0x3, TXPO = 0x1):\nTX = PAD2,\nRX = PAD3\n"
- moved on the sheet: C10, C11, C12, C13, C14, C15, C6, C7, C8, C9, L1

Commit message: fixed ERC failures
Connections:
- wire segments 67 -> 70
Changed lines of the file:
@@
 	5000 2600 5000 2500
 Wire Wire Line
-	5450 2500 5950 2500
+	5450 2500 5750 2500
 Connection ~ 5450 2500
 Wire Wire Line
@@
 Text Label 7150 4300 0    50   ~ 0
 SERCOM3.1_I2C_SCL
+$Comp
+L power:PWR_FLAG #FLG?
+U 1 1 5ECF1EAA
+P 5150 1650
+AR Path="/5ECF1EAA" Ref="#FLG?"  Part="1"
+AR Path="/5F3BBDAE/5ECF1EAA" Ref="#FLG0103"  Part="1"
+F 0 "#FLG0103" H 5150 1725 50  0001 C CNN
+F 1 "PWR_FLAG" V 5150 1777 50  0000 L CNN
+F 2 "" H 5150 1650 50  0001 C CNN
+F 3 "~" H 5150 1650 50  0001 C CNN
+	1    5150 1650
+	0    -1   -1   0
+$EndComp
+Wire Wire Line
+	5150 1650 5250 1650
+Connection ~ 5250 1650
+$Comp
+L power:PWR_FLAG #FLG?
+U 1 1 5ECF65DA
+P 5750 2600
+AR Path="/5ECF65DA" Ref="#FLG?"  Part="1"
+AR Path="/5F3BBDAE/5ECF65DA" Ref="#FLG0104"  Part="1"
+F 0 "#FLG0104" H 5750 2675 50  0001 C CNN
+F 1 "PWR_FLAG" V 5750 2727 50  0000 L CNN
+F 2 "" H 5750 2600 50  0001 C CNN
+F 3 "~" H 5750 2600 50  0001 C CNN
+	1    5750 2600
+	-1   0    0    1
+$EndComp
+Wire Wire Line
+	5750 2600 5750 2500
+Connection ~ 5750 2500
+Wire Wire Line
+	5750 2500 5950 2500
 $EndSCHEMATC

Commit message: added board layout, changed antenna connector.
Parts:
- C10, C11, C12, C13, C14, C15, C7, C8: footprint (none) -> Capacitor_SMD:C_1206_3216Metric_Pad1.42x1.75mm_HandSolder
- C6, C9: value C -> 18pF NPO; footprint (none) -> Capacitor_SMD:C_1206_3216Metric_Pad1.42x1.75mm_HandSolder
- FB1, L1: footprint (none) -> Inductor_SMD:L_0603_1608Metric_Pad1.05x0.95mm_HandSolder
- Y1: value MS1V-T1K -> MS1V-T1K 32mhz; footprint (none) -> Crystals:Crystal_SMD_TXC_9HT11-2pin_2.0x1.2mm_HandSoldering
Connections:
- wire segments 70 -> 72
Changed lines of the file:
@@
 EESchema Schematic File Version 4
-LIBS:board-cache
-EELAYER 29 0
+EELAYER 30 0
 EELAYER END
 $Descr A4 11693 8268
@@
 Text HLabel 4300 4400 0    50   BiDi ~ 0
 D0
-Text Label 3300 3150 0    50   ~ 0
-XOUT32
-Text Label 2800 3150 2    50   ~ 0
-XIN32
 Text Label 5150 3700 2    50   ~ 0
 XOUT32
@@
 F 0 "C8" H 3365 4496 50  0000 L CNN
 F 1 "100n" H 3365 4405 50  0000 L CNN
-F 2 "" H 3288 4300 50  0001 C CNN
+F 2 "Capacitor_SMD:C_1206_3216Metric_Pad1.42x1.75mm_HandSolder" H 3288 4300 50  0001 C CNN
 F 3 "~" H 3250 4450 50  0001 C CNN
 	1    3250 4450
@@
 F 0 "C7" H 2965 4496 50  0000 L CNN
 F 1 "4.7u" H 2965 4405 50  0000 L CNN
-F 2 "" H 2888 4300 50  0001 C CNN
+F 2 "Capacitor_SMD:C_1206_3216Metric_Pad1.42x1.75mm_HandSolder" H 2888 4300 50  0001 C CNN
 F 3 "~" H 2850 4450 50  0001 C CNN
 	1    2850 4450
@@
 	1    0    0    -1
 $EndComp
-Wire Wire Line
-	2800 3150 2900 3150
-Wire Wire Line
-	2800 3250 2800 3150
-Wire Wire Line
-	3300 3150 3200 3150
-Wire Wire Line
-	3300 3250 3300 3150
-$Comp
-L Device:C C?
-U 1 1 5F3C031F
-P 2800 3400
-AR Path="/5F3C031F" Ref="C?"  Part="1"
-AR Path="/5F3BBDAE/5F3C031F" Ref="C6"  Part="1"
-F 0 "C6" H 2686 3354 50  0000 R CNN
-F 1 "C" H 2686 3445 50  0000 R CNN
-F 2 "" H 2838 3250 50  0001 C CNN
-F 3 "~" H 2800 3400 50  0001 C CNN
-	1    2800 3400
-	1    0    0    1
-$EndComp
-$Comp
-L Device:C C?
-U 1 1 5F3C0319
-P 3300 3400
-AR Path="/5F3C0319" Ref="C?"  Part="1"
-AR Path="/5F3BBDAE/5F3C0319" Ref="C9"  Part="1"
-F 0 "C9" H 3185 3354 50  0000 R CNN
-F 1 "C" H 3185 3445 50  0000 R CNN
-F 2 "" H 3338 3250 50  0001 C CNN
-F 3 "~" H 3300 3400 50  0001 C CNN
-	1    3300 3400
-	-1   0    0    1
-$EndComp
-$Comp
-L Device:Crystal_GND2 Y?
-U 1 1 5F3C0313
-P 3050 3150
-AR Path="/5F3C0313" Ref="Y?"  Part="1"
-AR Path="/5F3BBDAE/5F3C0313" Ref="Y1"  Part="1"
-F 0 "Y1" H 3050 3418 50  0000 C CNN
-F 1 "MS1V-T1K" H 3050 3327 50  0000 C CNN
-F 2 "" H 3050 3150 50  0001 C CNN
-F 3 "~" H 3050 3150 50  0001 C CNN
-	1    3050 3150
-	1    0    0    -1
-$EndComp
 Text HLabel 4300 2500 0    50   Input ~ 0
 VDDIN
@@
 F 0 "C15" H 7065 2796 50  0000 L CNN
 F 1 "100n" H 7065 2705 50  0000 L CNN
-F 2 "" H 6988 2600 50  0001 C CNN
+F 2 "Capacitor_SMD:C_1206_3216Metric_Pad1.42x1.75mm_HandSolder" H 6988 2600 50  0001 C CNN
 F 3 "~" H 6950 2750 50  0001 C CNN
 	1    6950 2750
@@
 F 0 "C14" H 6665 2796 50  0000 L CNN
 F 1 "10u" H 6665 2705 50  0000 L CNN
-F 2 "" H 6588 2600 50  0001 C CNN
+F 2 "Capacitor_SMD:C_1206_3216Metric_Pad1.42x1.75mm_HandSolder" H 6588 2600 50  0001 C CNN
 F 3 "~" H 6550 2750 50  0001 C CNN
 	1    6550 2750
@@
 F 0 "C11" H 5565 1946 50  0000 L CNN
 F 1 "1u" H 5565 1855 50  0000 L CNN
-F 2 "" H 5488 1750 50  0001 C CNN
+F 2 "Capacitor_SMD:C_1206_3216Metric_Pad1.42x1.75mm_HandSolder" H 5488 1750 50  0001 C CNN
 F 3 "~" H 5450 1900 50  0001 C CNN
 	1    5450 1900
@@
 F 0 "FB1" V 4426 2500 50  0000 C CNN
 F 1 "FBMH3216HM221NT" V 4517 2500 50  0000 C CNN
-F 2 "" V 4630 2500 50  0001 C CNN
+F 2 "Inductor_SMD:L_0603_1608Metric_Pad1.05x0.95mm_HandSolder" V 4630 2500 50  0001 C CNN
 F 3 "~" H 4700 2500 50  0001 C CNN
 	1    4700 2500
@@
 F 0 "C13" H 5915 1946 50  0000 L CNN
 F 1 "100n" H 5915 1855 50  0000 L CNN
-F 2 "" H 5838 1750 50  0001 C CNN
+F 2 "Capacitor_SMD:C_1206_3216Metric_Pad1.42x1.75mm_HandSolder" H 5838 1750 50  0001 C CNN
 F 3 "~" H 5800 1900 50  0001 C CNN
 	1    5800 1900
@@
 F 0 "L1" H 6103 1696 50  0000 L CNN
 F 1 "10u" H 6103 1605 50  0000 L CNN
-F 2 "" H 6050 1650 50  0001 C CNN
+F 2 "Inductor_SMD:L_0603_1608Metric_Pad1.05x0.95mm_HandSolder" H 6050 1650 50  0001 C CNN
 F 3 "~" H 6050 1650 50  0001 C CNN
 	1    6050 1650
@@
 F 1 "ATSAML21E18B-AUT" H 6150 3850 50  0000 C CNN
 F 2 "Package_QFP:TQFP-32_7x7mm_P0.8mm" H 7150 5100 50  0001 C CNN
-F 3 "http://ww1.microchip.com/downloads/en/DeviceDoc/60001477A.pdf" H 6150 4200 50  0001 C CNN
+F 3 "http://ww1.microchip.com/downloads/en/DeviceDoc/SAM_L21_Family_DataSheet_DS60001477C.pdf" H 6150 4200 50  0001 C CNN
 	1    6150 4200
 	1    0    0    -1
@@
 F 0 "C12" H 5565 2796 50  0000 L CNN
 F 1 "100n" H 5565 2705 50  0000 L CNN
-F 2 "" H 5488 2600 50  0001 C CNN
+F 2 "Capacitor_SMD:C_1206_3216Metric_Pad1.42x1.75mm_HandSolder" H 5488 2600 50  0001 C CNN
 F 3 "~" H 5450 2750 50  0001 C CNN
 	1    5450 2750
@@
 F 0 "C10" H 5115 2796 50  0000 L CNN
 F 1 "10u" H 5115 2705 50  0000 L CNN
-F 2 "" H 5038 2600 50  0001 C CNN
+F 2 "Capacitor_SMD:C_1206_3216Metric_Pad1.42x1.75mm_HandSolder" H 5038 2600 50  0001 C CNN
 F 3 "~" H 5000 2750 50  0001 C CNN
 	1    5000 2750
@@
 Wire Wire Line
 	5750 2500 5950 2500
+Connection ~ 2800 3150
+Wire Wire Line
+	2800 3150 2650 3150
+Connection ~ 3300 3150
+Wire Wire Line
+	3300 3150 3450 3150
+$Comp
+L Device:Crystal_GND2 Y?
+U 1 1 5F3C0313
+P 3050 3150
+AR Path="/5F3C0313" Ref="Y?"  Part="1"
+AR Path="/5F3BBDAE/5F3C0313" Ref="Y1"  Part="1"
+F 0 "Y1" H 3050 3418 50  0000 C CNN
+F 1 "MS1V-T1K 32mhz" H 3050 3327 50  0000 C CNN
+F 2 "Crystals:Crystal_SMD_TXC_9HT11-2pin_2.0x1.2mm_HandSoldering" H 3050 3150 50  0001 C CNN
+F 3 "~" H 3050 3150 50  0001 C CNN
+	1    3050 3150
+	1    0    0    -1
+$EndComp
+$Comp
+L Device:C C?
+U 1 1 5F3C0319
+P 3300 3400
+AR Path="/5F3C0319" Ref="C?"  Part="1"
+AR Path="/5F3BBDAE/5F3C0319" Ref="C9"  Part="1"
+F 0 "C9" H 3185 3354 50  0000 R CNN
+F 1 "18pF NPO" H 3185 3445 50  0000 R CNN
+F 2 "Capacitor_SMD:C_1206_3216Metric_Pad1.42x1.75mm_HandSolder" H 3338 3250 50  0001 C CNN
+F 3 "~" H 3300 3400 50  0001 C CNN
+	1    3300 3400
+	-1   0    0    1
+$EndComp
+$Comp
+L Device:C C?
+U 1 1 5F3C031F
+P 2800 3400
+AR Path="/5F3C031F" Ref="C?"  Part="1"
+AR Path="/5F3BBDAE/5F3C031F" Ref="C6"  Part="1"
+F 0 "C6" H 2686 3354 50  0000 R CNN
+F 1 "18pF NPO" H 2686 3445 50  0000 R CNN
+F 2 "Capacitor_SMD:C_1206_3216Metric_Pad1.42x1.75mm_HandSolder" H 2838 3250 50  0001 C CNN
+F 3 "~" H 2800 3400 50  0001 C CNN
+	1    2800 3400
+	1    0    0    1
+$EndComp
+Wire Wire Line
+	3300 3250 3300 3150
+Wire Wire Line
+	3300 3150 3200 3150
+Wire Wire Line
+	2800 3250 2800 3150
+Wire Wire Line
+	2800 3150 2900 3150
+Text Label 2750 3150 2    50   ~ 0
+XIN32
+Text Label 3400 3150 0    50   ~ 0
+XOUT32
 $EndSCHEMATC
